File: board/board.kicad_pcb (KiCad board)
At the start: 2 copper layers, 21 x 13 mm, 1 part

Commit message: initial
Parts:
- added C1: 22uF, Capacitor_SMD:C_0805_2012Metric, F.Cu at (161.9, 102.0)
- added C10: 22uF, Capacitor_SMD:C_0805_2012Metric, F.Cu at (177.5, 98.3)
- added C11: 10pF, Capacitor_SMD:C_0402_1005Metric, F.Cu at (167.3, 92.9)
- added C12: 220nF, Capacitor_SMD:C_0402_1005Metric, F.Cu at (165.3, 92.0)
- added C13: 22uF, Capacitor_SMD:C_0805_2012Metric, F.Cu at (177.5, 96.3)
- added C14: 22uF, Capacitor_SMD:C_0805_2012Metric, F.Cu at (177.5, 94.3)
- added C15: 22uF, Capacitor_SMD:C_0805_2012Metric, F.Cu at (150.8, 95.5)
- added C16: 22uF, Capacitor_SMD:C_0805_2012Metric, F.Cu at (150.8, 97.5)
- added C17: 22uF, Capacitor_SMD:C_0805_2012Metric, F.Cu at (150.8, 93.5)
- added C18: 22uF, Capacitor_SMD:C_0805_2012Metric, F.Cu at (150.8, 91.5)
- added C2: 22uF, Capacitor_SMD:C_0805_2012Metric, F.Cu at (161.9, 100.0)
- added C3: 22uF, Capacitor_SMD:C_0805_2012Metric, F.Cu at (150.8, 99.5)
- added C4: 22uF, Capacitor_SMD:C_0805_2012Metric, F.Cu at (150.8, 101.5)
- added C5: 100nF, Capacitor_SMD:C_0402_1005Metric, F.Cu at (165.7, 99.7)
- added C6: 10pF, Capacitor_SMD:C_0402_1005Metric, F.Cu at (161.0, 92.8)
- added C7: 10nF, Capacitor_SMD:C_0402_1005Metric, F.Cu at (162.5, 92.3)
- added C8: 4.7nF, Capacitor_SMD:C_0402_1005Metric, F.Cu at (163.9, 91.7)
- added C9: 22uF, Capacitor_SMD:C_0805_2012Metric, F.Cu at (177.5, 100.3)
- added D1: SS12, Diode_SMD:D_SMA, F.Cu at (156.2, 94.3)
- added D2: SS12, Diode_SMD:D_SMA, F.Cu at (171.5, 94.3)
- added J1: Conn_01x02_Pin, Connector_PinHeader_2.54mm:PinHeader_1x02_P2.54mm_Vertical, F.Cu at (147.2, 92.3)
- added J2: Conn_01x02_Pin, Connector_PinHeader_2.54mm:PinHeader_1x02_P2.54mm_Vertical, F.Cu at (181.5, 96.1)
- added J3: 003_power, on_edge:on_edge_2x05_device, F.Cu at (140.0, 96.5)
- added L1: 4.7uH, Inductor_SMD:L_6.3x6.3_H3, F.Cu at (156.4, 99.5)
- added L2: 4.7uH, Inductor_SMD:L_6.3x6.3_H3, F.Cu at (171.7, 99.5)
- added NT1: NetTie_2, NetTie:NetTie-2_SMD_Pad0.5mm, F.Cu at (166.6, 98.8)
- added R1: 100R, Resistor_SMD:R_0603_1608Metric, F.Cu at (165.1, 101.0)
- added R2: 1M, Resistor_SMD:R_0402_1005Metric, F.Cu at (161.1, 93.7)
- added R3: 100k, Resistor_SMD:R_0402_1005Metric, F.Cu at (161.1, 91.8)
- added R5: 82k, Resistor_SMD:R_0402_1005Metric, F.Cu at (166.2, 92.9)
- added R6: 1M, Resistor_SMD:R_0402_1005Metric, F.Cu at (166.2, 91.1)
- added R7: 51k, Resistor_SMD:R_0402_1005Metric, F.Cu at (167.3, 91.1)
- added U1: TPS65131, Package_DFN_QFN:VQFN-24-1EP_4x4mm_P0.5mm_EP2.45x2.45mm_ThermalVias, F.Cu at (164.0, 95.9)
- LOGO1: moved to B.Cu
- moved LOGO1 6.40 mm to (156.3, 98.2), turned to 180 degrees
Routing:
- net GND: track 0.00 -> 38.7 mm, vias 0 -> 27
- net /DCDC/5V: track 0.00 -> 35.1 mm, vias 0 -> 4
- net /DCDC/-out: track 0.00 -> 26.7 mm
- net /DCDC/+out: track 0.00 -> 24.3 mm, vias 0 -> 1
- net Net-(D1-A): track 0.00 -> 17.9 mm
- net Net-(D2-K): track 0.00 -> 17.3 mm
- net /DCDC/GNDA: track 0.00 -> 16.1 mm, vias 0 -> 2
- net Net-(U1-ENN): track 0.00 -> 10.8 mm, vias 0 -> 2
- net Net-(U1-FBN): track 0.00 -> 4.79 mm
- net Net-(U1-FBP): track 0.00 -> 3.65 mm
- net Net-(U1-VREF): track 0.00 -> 3.12 mm
- net Net-(U1-CN): track 0.00 -> 2.02 mm
- net Net-(U1-CP): track 0.00 -> 1.68 mm
- net Net-(C11-Pad2): track 0.00 -> 0.87 mm
- added copper zone on B.Cu, net GND
- added copper zone on F.Cu, net GND
Other:
- board size 21 x 13 mm -> 45 x 13 mm
- board text added: "osf.000"
- board text added: "osf.b145.v1.0"
