File: board/board.kicad_pcb (KiCad board)
At the start: 2 copper layers, 45 x 13 mm, 34 parts, among them J1 Conn_01x02_Pin, J2 Conn_01x02_Pin, J3 003_power, U1 TPS65131

Commit message: initial b148
Parts:
- removed C1, C10, C13, C14, C15, C16, C17, C18, C2, C3, C4, C9: 22uF, Capacitor_SMD:C_0805_2012Metric
- removed C11, C6: 10pF, Capacitor_SMD:C_0402_1005Metric
- removed C12: 220nF, Capacitor_SMD:C_0402_1005Metric
- removed C5: 100nF, Capacitor_SMD:C_0402_1005Metric
- removed C7: 10nF, Capacitor_SMD:C_0402_1005Metric
- removed C8: 4.7nF, Capacitor_SMD:C_0402_1005Metric
- removed D1, D2: SS12, Diode_SMD:D_SMA
- removed J2: Conn_01x02_Pin, Connector_PinHeader_2.54mm:PinHeader_1x02_P2.54mm_Vertical
- removed J3: 003_power, on_edge:on_edge_2x05_device
- removed L1, L2: 4.7uH, Inductor_SMD:L_6.3x6.3_H3
- removed NT1: NetTie_2, NetTie:NetTie-2_SMD_Pad0.5mm
- removed R1: 100R, Resistor_SMD:R_0603_1608Metric
- removed R2, R6: 1M, Resistor_SMD:R_0402_1005Metric
- removed R3: 100k, Resistor_SMD:R_0402_1005Metric
- removed R5: 82k, Resistor_SMD:R_0402_1005Metric
- removed R7: 51k, Resistor_SMD:R_0402_1005Metric
- removed U1: TPS65131, Package_DFN_QFN:VQFN-24-1EP_4x4mm_P0.5mm_EP2.45x2.45mm_ThermalVias
- added RV1: 10k, Potentiometer_SMD:Potentiometer_Bourns_TC33X_Vertical, F.Cu at (147.8, 94.5)
- added RV2: 10k, Potentiometer_SMD:Potentiometer_Bourns_TC33X_Vertical, F.Cu at (155.7, 100.2)
- added RV3: 10k, Potentiometer_SMD:Potentiometer_Bourns_TC33X_Vertical, F.Cu at (147.8, 100.2)
- added RV4: 10k, Potentiometer_SMD:Potentiometer_Bourns_TC33X_Vertical, F.Cu at (155.7, 94.5)
- J1: value Conn_01x02_Pin -> 007_ADC; footprint Connector_PinHeader_2.54mm:PinHeader_1x02_P2.54mm_Vertical -> on_edge:on_edge_2x05_device
- moved J1 8.34 mm to (140.0, 96.5), turned to -90 degrees
- moved LOGO1 4.74 mm to (151.8, 99.3)
Connections:
- J1 pad 2: /DCDC/+out -> unconnected-(J1-VREF-Pad2)
Routing:
- net /DCDC/5V: track 35.1 -> 0.00 mm, vias 4 -> 0
- net Net-(J1-5V): track 0.00 -> 30.4 mm, vias 0 -> 1
- net /DCDC/-out: track 26.7 -> 0.00 mm
- net /DCDC/+out: track 24.3 -> 0.00 mm, vias 1 -> 0
- net Net-(D1-A): track 17.9 -> 0.00 mm
- net Net-(D2-K): track 17.3 -> 0.00 mm
- net /DCDC/GNDA: track 16.1 -> 0.00 mm, vias 2 -> 0
- net Net-(J1-ADC1): track 0.00 -> 14.0 mm
- net Net-(J1-ADC3): track 0.00 -> 13.9 mm, vias 0 -> 1
- net Net-(U1-ENN): track 10.8 -> 0.00 mm, vias 2 -> 0
- net GND: track 38.7 -> 29.6 mm, vias 27 -> 5
- net Net-(J1-ADC0): track 0.00 -> 6.90 mm
- net Net-(J1-ADC2): track 0.00 -> 6.15 mm
- net Net-(U1-FBN): track 4.79 -> 0.00 mm
- net Net-(U1-FBP): track 3.65 -> 0.00 mm
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Other:
- board size 45 x 13 mm -> 21 x 13 mm
- board text added: "osf.b148.v1.0"
- board text removed: "osf.000"
- board text removed: "osf.b145.v1.0"
